File: hardware/Dachshund60F/Dachshund60F.kicad_pcb (KiCad board)
At the start: 2 copper layers, 318.5 x 121.1 mm, 209 parts, among them J1 USB daughterboard (JST-SH 4P), J2 Battery (JST-PH 2P), J3 SWD, J4 Display, Q1 AO3401A, SW1 Power, SW100 MX Esc (1.00u), SW101 MX F1 (1.00u), SW102 MX F2 (1.00u), SW103 MX F3 (1.00u), SW104 MX F4 (1.00u), SW105 MX F5 (1.00u), SW106 MX F6 (1.00u), SW107 MX F7 (1.00u), SW108 MX F8 (1.00u), SW109 MX F9 (1.00u), SW110 MX F10 (1.00u), SW111 MX F11 (1.00u), SW112 MX F12 (1.00u), SW113 MX Delete (1.00u), SW2 Reset, SW200 MX ` (1.00u), SW201 MX 1 (1.00u), SW202 MX 2 (1.00u), SW203 MX 3 (1.00u), SW204 MX 4 (1.00u), SW205 MX 5 (1.00u), SW206 MX 6 (1.00u), SW207 MX 7 (1.00u), SW208 MX 8 (1.00u), SW209 MX 9 (1.00u), SW210 MX 0 (1.00u), SW211 MX - (1.00u), SW212 MX = (1.00u), SW213 MX Backspace (2.00u), SW3 PEC12R-4220F-S0024 (horizonta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, SW300 MX Tab (1.50u), SW301 MX Q (1.00u), SW302 MX W (1.00u), SW303 MX E (1.00u), SW304 MX R (1.00u), SW305 MX T (1.00u), SW306 MX Y (1.00u), SW307 MX U (1.00u), SW308 MX I (1.00u), SW309 MX O (1.00u), SW310 MX P (1.00u), SW311 MX [ (1.00u), SW312 MX ] (1.00u), SW313 MX \ (1.50u), SW400 MX Caps Lock (1.75u), SW401 MX A (1.00u), SW402 MX S (1.00u), SW403 MX D (1.00u), SW404 MX F (1.00u), SW405 MX G (1.00u), SW406 MX H (1.00u), SW407 MX J (1.00u), SW408 MX K (1.00u), SW409 MX L (1.00u), SW410 MX ; (1.00u), SW411 MX ' (1.00u), SW413 MX Enter (2.25u), SW500 MX Shift (2.25u), SW501 MX Z (1.00u), SW502 MX X (1.00u), SW503 MX C (1.00u), SW504 MX V (1.00u), SW505 MX B (1.00u), SW506 MX N (1.00u), SW507 MX M (1.00u), SW508 MX , (1.00u), SW509 MX . (1.00u), SW510 MX / (1.00u), SW512 MX Shift (1.75u), SW513 MX Up (1.00u), SW600 MX Ctrl (1.25u), SW601 MX Win (1.25u), SW603 MX Alt (1.25u), SW604 MX Mod (1.25u, solder)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

Commit message: Add test pads for probing the mainboard
Nine 1.5 mm SMD test pads on the back, each on its net's existing
track with the net name on the silkscreen: VBUS, VBAT, VBAT_SW, VSYS,
+3V3, LED_VDD, CHG_STAT and two GND. Excluded from the BOM. DRC and ERC
show no new errors or warnings. The bring-up plan lists where each is.

Co-Authored-By: Claude Opus 5.5 (1M context) <noreply@anthropic.com>
Claude-Session: https://claude.ai/code/session_01D9WgQVzjyM3BLJSpari9iy
Parts:
- added TP1: VBUS, TestPoint:TestPoint_Pad_D1.5mm, B.Cu at (325.6, 89.2)
- added TP2: VBAT, TestPoint:TestPoint_Pad_D1.5mm, B.Cu at (322.0, 93.2)
- added TP3: VBAT_SW, TestPoint:TestPoint_Pad_D1.5mm, B.Cu at (331.5, 110.5)
- added TP4: VSYS, TestPoint:TestPoint_Pad_D1.5mm, B.Cu at (323.1, 116.0)
- added TP5: +3V3, TestPoint:TestPoint_Pad_D1.5mm, B.Cu at (318.2, 110.4)
- added TP6: LED_VDD, TestPoint:TestPoint_Pad_D1.5mm, B.Cu at (314.6, 123.4)
- added TP7: CHG_STAT, TestPoint:TestPoint_Pad_D1.5mm, B.Cu at (308.4, 71.5)
- added TP8: GND, TestPoint:TestPoint_Pad_D1.5mm, B.Cu at (321.5, 96.5)
- added TP9: GND, TestPoint:TestPoint_Pad_D1.5mm, B.Cu at (319.5, 120.5)
Routing:
- net GND: vias 648 -> 641

Commit message: Mainboard: lower the charge current to 300 mA (R1 = 3.3 kΩ)
The 500 mA charge current plus the keyboard's own load through D8
came to about 630 mA, over a 500 mA USB port's budget (project review
finding H1). R1 sets I = 1000 V / R_PROG, so 3.3 kΩ gives about 300 mA.
Value change only, in the schematic and the PCB; the bring-up plan's
charger numbers follow.

Co-Authored-By: Claude Opus 5.5 (1M context) <noreply@anthropic.com>
Claude-Session: https://claude.ai/code/session_01La3JB4NYHq7NgWrfFS2bsw
Parts:
- R1: value 2k -> 3.3k
Changed lines of the file:
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@@
 			)
 		)
-		(property "Value" "2k"
+		(property "Value" "3.3k"
 			(at 0 -1.43 90)
 			(unlocked yes)
