File: hardware/Dachshund60F/Dachshund60F.kicad_pcb (KiCad board)
At the start: 2 copper layers, 318.5 x 121.1 mm, 218 parts, among them J1 USB daughterboard (JST-SH 4P), J2 Battery (JST-PH 2P), J3 SWD, J4 Display, Q1 AO3401A, SW1 Power, SW100 MX Esc (1.00u), SW101 MX F1 (1.00u), SW102 MX F2 (1.00u), SW103 MX F3 (1.00u), SW104 MX F4 (1.00u), SW105 MX F5 (1.00u), SW106 MX F6 (1.00u), SW107 MX F7 (1.00u), SW108 MX F8 (1.00u), SW109 MX F9 (1.00u), SW110 MX F10 (1.00u), SW111 MX F11 (1.00u), SW112 MX F12 (1.00u), SW113 MX Delete (1.00u), SW2 Reset, SW200 MX ` (1.00u), SW201 MX 1 (1.00u), SW202 MX 2 (1.00u), SW203 MX 3 (1.00u), SW204 MX 4 (1.00u), SW205 MX 5 (1.00u), SW206 MX 6 (1.00u), SW207 MX 7 (1.00u), SW208 MX 8 (1.00u), SW209 MX 9 (1.00u), SW210 MX 0 (1.00u), SW211 MX - (1.00u), SW212 MX = (1.00u), SW213 MX Backspace (2.00u), SW3 PEC12R-4220F-S0024 (horizonta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, SW300 MX Tab (1.50u), SW301 MX Q (1.00u), SW302 MX W (1.00u), SW303 MX E (1.00u), SW304 MX R (1.00u), SW305 MX T (1.00u), SW306 MX Y (1.00u), SW307 MX U (1.00u), SW308 MX I (1.00u), SW309 MX O (1.00u), SW310 MX P (1.00u), SW311 MX [ (1.00u), SW312 MX ] (1.00u), SW313 MX \ (1.50u), SW400 MX Caps Lock (1.75u), SW401 MX A (1.00u), SW402 MX S (1.00u), SW403 MX D (1.00u), SW404 MX F (1.00u), SW405 MX G (1.00u), SW406 MX H (1.00u), SW407 MX J (1.00u), SW408 MX K (1.00u), SW409 MX L (1.00u), SW410 MX ; (1.00u), SW411 MX ' (1.00u), SW413 MX Enter (2.25u), SW500 MX Shift (2.25u), SW501 MX Z (1.00u), SW502 MX X (1.00u), SW503 MX C (1.00u), SW504 MX V (1.00u), SW505 MX B (1.00u), SW506 MX N (1.00u), SW507 MX M (1.00u), SW508 MX , (1.00u), SW509 MX . (1.00u), SW510 MX / (1.00u), SW512 MX Shift (1.75u), SW513 MX Up (1.00u), SW600 MX Ctrl (1.25u), SW601 MX Win (1.25u), SW603 MX Alt (1.25u), SW604 MX Mod (1.25u, solder)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

Commit message: SW3: PEC12R-2220F-S0024, the shaft-parallel part
PEC12R-4220F-S0024 is Bourns' horizontal-mount part, whose shaft stands
up from the board. The roller needs the vertical-mount (radial pin) part,
which the footprint is drawn for. Tiam chose 24 detents: PEC12R-2220F-S0024
(20 mm shaft, push switch, 24 pulses). Update the schematic value, MPN and
LCSC number (C49673168), the PCB value and the docs.

Co-Authored-By: Claude Opus 5.5 (1M context) <noreply@anthropic.com>
Parts:
- SW3: value PEC12R-4220F-S0024 (horizontal, 20 mm shaft) -> PEC12R-2220F-S0024 (shaft parallel to the board, 20 mm)
Changed lines of the file:
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@@
 			)
 		)
-		(property "Value" "PEC12R-4220F-S0024 (horizontal, 20 mm shaft)"
+		(property "Value" "PEC12R-2220F-S0024 (shaft parallel to the board, 20 mm)"
 			(at 0 12 180)
 			(unlocked yes)

Commit message: SW3: the 30 mm shaft, PEC12R-2230F-S0024
Tiam chose the 30 mm shaft so the wheel that reaches out through the end
wall sits on about 19 mm of shaft. Update the schematic value and MPN (LCSC
has no listing, so the LCSC field is cleared), the PCB value and the docs.
gen_models.py takes the shaft length as a parameter and builds the 30 mm
model (tip at board x 340.8, 12 mm D-flat); SW3 uses it. Refresh the
mainboard and assembly STEP.

Co-Authored-By: Claude Opus 5.5 (1M context) <noreply@anthropic.com>
Parts:
- SW3: value PEC12R-2220F-S0024 (shaft parallel to the board, 20 mm) -> PEC12R-2230F-S0024 (shaft parallel to the board, 30 mm)
Changed lines of the file:
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@@
 			)
 		)
-		(property "Value" "PEC12R-2220F-S0024 (shaft parallel to the board, 20 mm)"
+		(property "Value" "PEC12R-2230F-S0024 (shaft parallel to the board, 30 mm)"
 			(at 0 12 180)
 			(unlocked yes)
@@
 		)
 		(embedded_fonts no)
-		(model "${KIPRJMOD}/../3dmodels/Bourns_PEC12R-2x20F-S_standin.step"
+		(model "${KIPRJMOD}/../3dmodels/Bourns_PEC12R-2x30F-S_standin.step"
 			(offset
 				(xyz 0 0 0)
