File: hardware/Dachshund60F/Dachshund60F.kicad_sch (KiCad schematic)
At the start: 218 parts, among them J1 USB daughterboard (JST-SH 4P), J2 Battery (JST-PH 2P), J3 SWD, J4 Display, Q1 AO3401A, SW1 Power, SW100 MX Esc (1.00u), SW101 MX F1 (1.00u), SW102 MX F2 (1.00u), SW103 MX F3 (1.00u), SW104 MX F4 (1.00u), SW105 MX F5 (1.00u), SW106 MX F6 (1.00u), SW107 MX F7 (1.00u), SW108 MX F8 (1.00u), SW109 MX F9 (1.00u), SW110 MX F10 (1.00u), SW111 MX F11 (1.00u), SW112 MX F12 (1.00u), SW113 MX Delete (1.00u), SW2 Reset, SW200 MX ` (1.00u), SW201 MX 1 (1.00u), SW202 MX 2 (1.00u), SW203 MX 3 (1.00u), SW204 MX 4 (1.00u), SW205 MX 5 (1.00u), SW206 MX 6 (1.00u), SW207 MX 7 (1.00u), SW208 MX 8 (1.00u), SW209 MX 9 (1.00u), SW210 MX 0 (1.00u), SW211 MX - (1.00u), SW212 MX = (1.00u), SW213 MX Backspace (2.00u), SW3 PEC12R-4220F-S0024 (horizonta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, SW300 MX Tab (1.50u), SW301 MX Q (1.00u), SW302 MX W (1.00u), SW303 MX E (1.00u), SW304 MX R (1.00u), SW305 MX T (1.00u), SW306 MX Y (1.00u), SW307 MX U (1.00u), SW308 MX I (1.00u), SW309 MX O (1.00u), SW310 MX P (1.00u), SW311 MX [ (1.00u), SW312 MX ] (1.00u), SW313 MX \ (1.50u), SW400 MX Caps Lock (1.75u), SW401 MX A (1.00u), SW402 MX S (1.00u), SW403 MX D (1.00u), SW404 MX F (1.00u), SW405 MX G (1.00u), SW406 MX H (1.00u), SW407 MX J (1.00u), SW408 MX K (1.00u), SW409 MX L (1.00u), SW410 MX ; (1.00u), SW411 MX ' (1.00u), SW413 MX Enter (2.25u), SW500 MX Shift (2.25u), SW501 MX Z (1.00u), SW502 MX X (1.00u), SW503 MX C (1.00u), SW504 MX V (1.00u), SW505 MX B (1.00u), SW506 MX N (1.00u), SW507 MX M (1.00u), SW508 MX , (1.00u), SW509 MX . (1.00u), SW510 MX / (1.00u), SW512 MX Shift (1.75u), SW513 MX Up (1.00u), SW600 MX Ctrl (1.25u), SW601 MX Win (1.25u), SW603 MX Alt (1.25u), SW604 MX Mod (1.25u, solder)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

Commit message: Mainboard: lower the charge current to 300 mA (R1 = 3.3 kΩ)
The 500 mA charge current plus the keyboard's own load through D8
came to about 630 mA, over a 500 mA USB port's budget (project review
finding H1). R1 sets I = 1000 V / R_PROG, so 3.3 kΩ gives about 300 mA.
Value change only, in the schematic and the PCB; the bring-up plan's
charger numbers follow.

Co-Authored-By: Claude Opus 5.5 (1M context) <noreply@anthropic.com>
Claude-Session: https://claude.ai/code/session_01La3JB4NYHq7NgWrfFS2bsw
Parts:
- R1: value 2k -> 3.3k
Changed lines of the file:
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@@
 			)
 		)
-		(property "Value" "2k"
+		(property "Value" "3.3k"
 			(at 55.88 228.6 90)
 			(effects

Commit message: JLCPCB assembly: LCSC and MPN fields on every assembled part, BOM and CPL export
Every part JLC assembles on the mainboard, daughterboard and dongle now has
an LCSC number checked on jlcpcb.com, including the Kailh hot-swap sockets.
export_fab.py writes JLC-format BOM and CPL files and moves the sockets to the
bottom layer at their own centre. F1 becomes BHFUSE BSMD1206-075-6V (same
1206 / 750 mA rating as MF-NSMF075-2, which LCSC doesn't stock).

Co-Authored-By: Claude Opus 5.5 (1M context) <noreply@anthropic.com>
Claude-Session: https://claude.ai/code/session_01P5t8x38EvinT9rpFK5k2Rj
Parts:
- C1, C2, C3, C4, C6: LCSC (none) -> C19666; MPN (none) -> Samsung CL10A475KO8NNNC
- C10, C11: LCSC (none) -> C15195; MPN (none) -> Samsung CL05B103KB5NNNC
- C12: LCSC (none) -> C52923; MPN (none) -> Samsung CL05A105KA5NQNC
- C13, C14, C15, C16, C17, C18, C19, C5, C7: LCSC (none) -> C1525; MPN (none) -> Samsung CL05B104KO5NNNC
- C8, C9: LCSC (none) -> C1547; MPN (none) -> FH 0402CG120J500NT
- D1: LCSC (none) -> C2991936; MPN (none) -> CJ BAT54WS
- D100, D101, D102, D103, D104, D105, D106, D107, D108, D109, D110, D111, D112, D113, D114, D200, D201, D202, D203, D204, D205, D206, D207, D208, D209, D210, D211, D212, D213, D300, D301, D302, D303, D304, D305, D306, D307, D308, D309, D310, D311, D312, D313, D400, D401, D402, D403, D404, D405, D406, D407, D408, D409, D410, D411, D413, D500, D501, D502, D503, D504, D505, D506, D507, D508, D509, D510, D512, D513, D600, D601, D603, D604, D606, D608, D610, D611, D612, D613, D614: LCSC (none) -> C81598; MPN (none) -> 1N4148W
- D2, D3, D4, D5, D6, D7: LCSC (none) -> C5149201; MPN (none) -> OPSCO SK6812MINI-E
- D8: LCSC (none) -> C8598; MPN (none) -> B5819W SL
- J1: LCSC (none) -> C160404; MPN (none) -> JST SM04B-SRSS-TB(LF)(SN)
- J2: LCSC (none) -> C295747; MPN (none) -> JST S2B-PH-SM4-TB(LF)(SN)
- J3: LCSC (none) -> C962329; MPN (none) -> XFCN PZ127V-11-05-H25
- Q1: LCSC (none) -> C15127; MPN (none) -> AO3401A
- R1: LCSC (none) -> C22978; MPN (none) -> UNI-ROYAL 0603WAF3301T5E
- R2: LCSC (none) -> C25741; MPN (none) -> UNI-ROYAL 0402WGF1003TCE
- R3: LCSC (none) -> C25803; MPN (none) -> UNI-ROYAL 0603WAF1003T5E
- SW1: LCSC (none) -> C221841; MPN (none) -> C&K PCM12SMTR
- SW100, SW101, SW102, SW103, SW104, SW105, SW106, SW107, SW108, SW109, SW110, SW111, SW112, SW113, SW200, SW201, SW202, SW203, SW204, SW205, SW206, SW207, SW208, SW209, SW210, SW211, SW212, SW213, SW300, SW301, SW302, SW303, SW304, SW305, SW306, SW307, SW308, SW309, SW310, SW311, SW312, SW313, SW400, SW401, SW402, SW403, SW404, SW405, SW406, SW407, SW408, SW409, SW410, SW411, SW413, SW500, SW501, SW502, SW503, SW504, SW505, SW506, SW507, SW508, SW509, SW510, SW512, SW513, SW600, SW601, SW603, SW608, SW610, SW611, SW612, SW613, SW614: LCSC (none) -> C2803348; MPN (none) -> Kailh CPG151101S11 (hot-swap socket; switch not included)
- SW2: LCSC (none) -> C2886898; MPN (none) -> E-Switch TL3342F160QG
- SW3: LCSC (none) -> C18164805; MPN (none) -> Bourns PEC12R-4220F-S0024
- U1: LCSC (none) -> C5118826; MPN (none) -> Raytac MDBT50Q-1MV2
- U2: LCSC (none) -> C424093; MPN (none) -> Microchip MCP73831T-2ACI/OT
- U3: LCSC (none) -> C2681320; MPN (none) -> TI TPS22917DBVR
- U4: LCSC (none) -> C100024; MPN (none) -> TI SN74LV1T34DBVR
- Y1: LCSC (none) -> C255869; MPN (none) -> Epson X1A0000910005 (32.768 kHz, 9 pF)

Commit message: Mainboard BOM: hot-swap sockets to HanElectricity CPG151101S11-2 (C49352235)
JLC has no stock of the Kailh CPG151101S11 (C2803348). The -2's datasheet
matches the Kailh socket and the footprint (6.35 x 2.54 mm hole spacing,
3.0 mm holes, 2.55 x 2.5 mm pads, 14.5 x 5.89 x 1.85 mm body).

Co-Authored-By: Claude Opus 5.5 <noreply@anthropic.com>
Claude-Session: https://claude.ai/code/session_01P5t8x38EvinT9rpFK5k2Rj
Parts:
- SW100, SW101, SW102, SW103, SW104, SW105, SW106, SW107, SW108, SW109, SW110, SW111, SW112, SW113, SW200, SW201, SW202, SW203, SW204, SW205, SW206, SW207, SW208, SW209, SW210, SW211, SW212, SW213, SW300, SW301, SW302, SW303, SW304, SW305, SW306, SW307, SW308, SW309, SW310, SW311, SW312, SW313, SW400, SW401, SW402, SW403, SW404, SW405, SW406, SW407, SW408, SW409, SW410, SW411, SW413, SW500, SW501, SW502, SW503, SW504, SW505, SW506, SW507, SW508, SW509, SW510, SW512, SW513, SW600, SW601, SW603, SW608, SW610, SW611, SW612, SW613, SW614: LCSC C2803348 -> C49352235; MPN Kailh CPG151101S11 (hot-swap socket; switch not included) -> HanElectricity CPG151101S11-2 (Kailh-pattern hot-swap socke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

Commit message: Use the MDBT50Q-P1MV2 module on the keyboard and dongle
The -P1MV2 is the same Raytac nRF52840 module with a PCB trace antenna
instead of a chip antenna: same 15.5 x 10.5 mm body, same 61 pads,
antenna at the same end. Footprint and keep-outs are unchanged; only
the Value, MPN and LCSC (C5119772) fields and the docs change. It costs
about C$10.74 at JLC against C$25.71, for about 20 % less rated
open-air range.

Co-Authored-By: Claude Opus 5.5 <noreply@anthropic.com>
Claude-Session: https://claude.ai/code/session_01P5t8x38EvinT9rpFK5k2Rj
Parts:
- U1: value MDBT50Q-1MV2 -> MDBT50Q-P1MV2; LCSC C5118826 -> C5119772; MPN Raytac MDBT50Q-1MV2 -> Raytac MDBT50Q-P1MV2
Changed lines of the file:
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@@
 			)
 		)
-		(property "Value" "MDBT50Q-1MV2"
+		(property "Value" "MDBT50Q-P1MV2"
 			(at 80.01 123.19 0)
 			(effects
@@
 			)
 		)
-		(property "MPN" "Raytac MDBT50Q-1MV2"
+		(property "MPN" "Raytac MDBT50Q-P1MV2"
 			(at 80.01 123.19 0)
 			(hide yes)
@@
 			)
 		)
-		(property "LCSC" "C5118826"
+		(property "LCSC" "C5119772"
 			(at 80.01 123.19 0)
 			(hide yes)

Commit message: SW3: PEC12R-2220F-S0024, the shaft-parallel part
PEC12R-4220F-S0024 is Bourns' horizontal-mount part, whose shaft stands
up from the board. The roller needs the vertical-mount (radial pin) part,
which the footprint is drawn for. Tiam chose 24 detents: PEC12R-2220F-S0024
(20 mm shaft, push switch, 24 pulses). Update the schematic value, MPN and
LCSC number (C49673168), the PCB value and the docs.

Co-Authored-By: Claude Opus 5.5 (1M context) <noreply@anthropic.com>
Parts:
- SW3: value PEC12R-4220F-S0024 (horizontal, 20 mm shaft) -> PEC12R-2220F-S0024 (shaft parallel to the board, 20 mm); LCSC C18164805 -> C49673168; MPN Bourns PEC12R-4220F-S0024 -> Bourns PEC12R-2220F-S0024
Changed lines of the file:
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@@
 			)
 		)
-		(property "Value" "PEC12R-4220F-S0024 (horizontal, 20 mm shaft)"
+		(property "Value" "PEC12R-2220F-S0024 (shaft parallel to the board, 20 mm)"
 			(at 30.48 323.85 0)
 			(effects
@@
 			)
 		)
-		(property "MPN" "Bourns PEC12R-4220F-S0024"
+		(property "MPN" "Bourns PEC12R-2220F-S0024"
 			(at 30.48 323.85 0)
 			(hide yes)
@@
 			)
 		)
-		(property "LCSC" "C18164805"
+		(property "LCSC" "C49673168"
 			(at 30.48 323.85 0)
 			(hide yes)

Commit message: SW3: the 30 mm shaft, PEC12R-2230F-S0024
Tiam chose the 30 mm shaft so the wheel that reaches out through the end
wall sits on about 19 mm of shaft. Update the schematic value and MPN (LCSC
has no listing, so the LCSC field is cleared), the PCB value and the docs.
gen_models.py takes the shaft length as a parameter and builds the 30 mm
model (tip at board x 340.8, 12 mm D-flat); SW3 uses it. Refresh the
mainboard and assembly STEP.

Co-Authored-By: Claude Opus 5.5 (1M context) <noreply@anthropic.com>
Parts:
- SW3: value PEC12R-2220F-S0024 (shaft parallel to the board, 20 mm) -> PEC12R-2230F-S0024 (shaft parallel to the board, 30 mm); LCSC C49673168 -> (none); MPN Bourns PEC12R-2220F-S0024 -> Bourns PEC12R-2230F-S0024
Changed lines of the file:
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@@
 			)
 		)
-		(property "Value" "PEC12R-2220F-S0024 (shaft parallel to the board, 20 mm)"
+		(property "Value" "PEC12R-2230F-S0024 (shaft parallel to the board, 30 mm)"
 			(at 30.48 323.85 0)
 			(effects
@@
 			)
 		)
-		(property "MPN" "Bourns PEC12R-2220F-S0024"
+		(property "MPN" "Bourns PEC12R-2230F-S0024"
 			(at 30.48 323.85 0)
 			(hide yes)
@@
 			)
 		)
-		(property "LCSC" "C49673168"
+		(property "LCSC" ""
 			(at 30.48 323.85 0)
 			(hide yes)
