File: hardware/Dachshund60F-USB/Dachshund60F-USB.kicad_sch (KiCad schematic)
At the start: 9 parts, among them J1 USB-C (HRO TYPE-C-31-M-12), J2 Mainboard (JST-SH 4P), U1 USBLC6-2SC6

Commit message: JLCPCB assembly: LCSC and MPN fields on every assembled part, BOM and CPL export
Every part JLC assembles on the mainboard, daughterboard and dongle now has
an LCSC number checked on jlcpcb.com, including the Kailh hot-swap sockets.
export_fab.py writes JLC-format BOM and CPL files and moves the sockets to the
bottom layer at their own centre. F1 becomes BHFUSE BSMD1206-075-6V (same
1206 / 750 mA rating as MF-NSMF075-2, which LCSC doesn't stock).

Co-Authored-By: Claude Opus 5.5 (1M context) <noreply@anthropic.com>
Claude-Session: https://claude.ai/code/session_01P5t8x38EvinT9rpFK5k2Rj
Parts:
- F1: LCSC (none) -> C883127; MPN Bourns MF-NSMF075-2 -> BHFUSE BSMD1206-075-6V
- FB1: LCSC (none) -> C1017
Changed lines of the file:
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@@
+			)
+		)
+		(property "LCSC" "C883127"
+			(at 142.24 67.31 0)
+			(hide yes)
+			(effects
+				(font
+					(size 1.27 1.27)
+				)
 			)
 		)
@@
 			)
 		)
-		(property "MPN" "Bourns MF-NSMF075-2"
+		(property "MPN" "BHFUSE BSMD1206-075-6V"
 			(at 139.7 63.5 0)
 			(hide yes)
@@
 			)
 		)
+		(property "LCSC" "C1017"
+			(at 78.74 146.05 0)
+			(hide yes)
+			(effects
+				(font
+					(size 1.27 1.27)
+				)
+			)
+		)
