File: hardware/Dachshund60F-Dongle/Dachshund60F-Dongle.kicad_pcb (KiCad board)
At the start: 2 copper layers, 40 x 24 mm, 20 parts, among them J1 USB-C (HRO TYPE-C-31-M-12), J2 SWD, SW1 Pair, SW2 Reset, U1 USBLC6-2SC6, U2 MDBT50Q-1MV2

Commit message: Use the MDBT50Q-P1MV2 module on the keyboard and dongle
The -P1MV2 is the same Raytac nRF52840 module with a PCB trace antenna
instead of a chip antenna: same 15.5 x 10.5 mm body, same 61 pads,
antenna at the same end. Footprint and keep-outs are unchanged; only
the Value, MPN and LCSC (C5119772) fields and the docs change. It costs
about C$10.74 at JLC against C$25.71, for about 20 % less rated
open-air range.

Co-Authored-By: Claude Opus 5.5 <noreply@anthropic.com>
Claude-Session: https://claude.ai/code/session_01P5t8x38EvinT9rpFK5k2Rj
Parts:
- U2: value MDBT50Q-1MV2 -> MDBT50Q-P1MV2
Changed lines of the file:
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@@
 			)
 		)
-		(property "Value" "MDBT50Q-1MV2"
+		(property "Value" "MDBT50Q-P1MV2"
 			(at 0.2 8.95 270)
 			(layer "F.Fab")
@@
 			)
 		)
-		(property "MPN" "Raytac MDBT50Q-1MV2"
+		(property "MPN" "Raytac MDBT50Q-P1MV2"
 			(at 0 0 270)
 			(layer "F.Fab")
