File: hardware/Dachshund60F-Dongle/Dachshund60F-Dongle.kicad_sch (KiCad schematic)
At the start: 20 parts, among them J1 USB-C (HRO TYPE-C-31-M-12), J2 SWD, SW1 Pair, SW2 Reset, U1 USBLC6-2SC6, U2 MDBT50Q-1MV2

Commit message: JLCPCB assembly: LCSC and MPN fields on every assembled part, BOM and CPL export
Every part JLC assembles on the mainboard, daughterboard and dongle now has
an LCSC number checked on jlcpcb.com, including the Kailh hot-swap sockets.
export_fab.py writes JLC-format BOM and CPL files and moves the sockets to the
bottom layer at their own centre. F1 becomes BHFUSE BSMD1206-075-6V (same
1206 / 750 mA rating as MF-NSMF075-2, which LCSC doesn't stock).

Co-Authored-By: Claude Opus 5.5 (1M context) <noreply@anthropic.com>
Claude-Session: https://claude.ai/code/session_01P5t8x38EvinT9rpFK5k2Rj
Parts:
- C1, C3: LCSC (none) -> C19666
- C2, C4: LCSC (none) -> C1525
- F1: LCSC (none) -> C883127; MPN Bourns MF-NSMF075-2 -> BHFUSE BSMD1206-075-6V
- FB1: LCSC (none) -> C1017
- J2: LCSC (none) -> C962329; MPN (none) -> XFCN PZ127V-11-05-H25
- R3: LCSC (none) -> C11702
- R4, R5: LCSC (none) -> C25104
- SW1, SW2: LCSC (none) -> C2886898
- U2: LCSC (none) -> C5118826
Changed lines of the file:
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@@
+			)
+		)
+		(property "LCSC" "C883127"
+			(at 86.36 69.85 0)
+			(hide yes)
+			(effects
+				(font
+					(size 1.27 1.27)
+				)
 			)
 		)
@@
 			)
 		)
-		(property "MPN" "Bourns MF-NSMF075-2"
+		(property "MPN" "BHFUSE BSMD1206-075-6V"
 			(at 83.82 66.04 0)
 			(hide yes)
@@
 			)
 		)
+		(property "LCSC" "C1017"
+			(at 104.14 140.97 0)
+			(hide yes)
+			(effects
+				(font
+					(size 1.27 1.27)
+				)
+			)
+		)
 		(property "Footprint" "Inductor_SMD:L_0805_2012Metric"
 			(at 101.6 137.16 0)
@@
 			)
 		)
+		(property "LCSC" "C5118826"
+			(at 154.94 55.88 0)
+			(hide yes)
+			(effects
+				(font
+					(size 1.27 1.27)
+				)
+			)
+		)
 		(property "Footprint" "RF_Module:Raytac_MDBT50Q"
 			(at 162.56 104.14 0)
@@
 			)
 		)
+		(property "LCSC" "C19666"
+			(at 213.36 64.77 0)
+			(hide yes)
+			(effects
+				(font
+					(size 1.27 1.27)
+				)
+			)
+		)
 		(property "Footprint" "Capacitor_SMD:C_0603_1608Metric"
 			(at 210.82 60.96 0)
@@
 			)
 		)
+		(property "LCSC" "C1525"
+			(at 223.52 64.77 0)
+			(hide yes)
+			(effects
+				(font
+					(size 1.27 1.27)
+				)
+			)
+		)
 		(property "Footprint" "Capacitor_SMD:C_0402_1005Metric"
 			(at 220.98 60.96 0)
@@
 			)
 		)
+		(property "LCSC" "C19666"
+			(at 238.76 64.77 0)
+			(hide yes)
+			(effects
+				(font
+					(size 1.27 1.27)
+				)
+			)
+		)
 		(property "Footprint" "Capacitor_SMD:C_0603_1608Metric"
 			(at 236.22 60.96 0)
@@
 			)
 		)
+		(property "LCSC" "C1525"
+			(at 248.92 64.77 0)
+			(hide yes)
+			(effects
+				(font
+					(size 1.27 1.27)
+				)
+			)
+		)
 		(property "Footprint" "Capacitor_SMD:C_0402_1005Metric"
 			(at 246.38 60.96 0)
@@
 			)
 		)
+		(property "LCSC" "C11702"
+			(at 236.22 105.41 0)
+			(hide yes)
+			(effects
+				(font
+					(size 1.27 1.27)
+				)
+			)
+		)
 		(property "Footprint" "Resistor_SMD:R_0402_1005Metric"
 			(at 233.68 101.6 0)
@@
 			)
 		)
+		(property "LCSC" "C25104"
+			(at 246.38 105.41 0)
+			(hide yes)
+			(effects
+				(font
+					(size 1.27 1.27)
+				)
+			)
+		)
 		(property "Footprint" "Resistor_SMD:R_0402_1005Metric"
 			(at 243.84 101.6 0)
@@
 			)
 		)
+		(property "LCSC" "C25104"
+			(at 256.54 105.41 0)
+			(hide yes)
+			(effects
+				(font
+					(size 1.27 1.27)
+				)
+			)
+		)
 		(property "Footprint" "Resistor_SMD:R_0402_1005Metric"
 			(at 254 101.6 0)
@@
 			)
 		)
+		(property "LCSC" "C2886898"
+			(at 215.9 156.21 0)
+			(hide yes)
+			(effects
+				(font
+					(size 1.27 1.27)
+				)
+			)
+		)
 		(property "Footprint" "Button_Switch_SMD:SW_SPST_TL3342"
 			(at 213.36 152.4 0)
@@
 			)
 		)
+		(property "LCSC" "C2886898"
+			(at 246.38 156.21 0)
+			(hide yes)
+			(effects
+				(font
+					(size 1.27 1.27)
+				)
+			)
+		)
 		(property "Footprint" "Button_Switch_SMD:SW_SPST_TL3342"
 			(at 243.84 152.4 0)
@@
 			)
 		)
+		(property "MPN" "XFCN PZ127V-11-05-H25"
+			(at 261.62 116.84 0)
+			(hide yes)
+			(effects
+				(font
+					(size 1.27 1.27)
+				)
+			)
+		)
+		(property "LCSC" "C962329"
+			(at 261.62 116.84 0)
+			(hide yes)
+			(effects
+				(font
+					(size 1.27 1.27)
+				)
+			)
+		)

Commit message: Use the MDBT50Q-P1MV2 module on the keyboard and dongle
The -P1MV2 is the same Raytac nRF52840 module with a PCB trace antenna
instead of a chip antenna: same 15.5 x 10.5 mm body, same 61 pads,
antenna at the same end. Footprint and keep-outs are unchanged; only
the Value, MPN and LCSC (C5119772) fields and the docs change. It costs
about C$10.74 at JLC against C$25.71, for about 20 % less rated
open-air range.

Co-Authored-By: Claude Opus 5.5 <noreply@anthropic.com>
Claude-Session: https://claude.ai/code/session_01P5t8x38EvinT9rpFK5k2Rj
Parts:
- U2: value MDBT50Q-1MV2 -> MDBT50Q-P1MV2; LCSC C5118826 -> C5119772; MPN Raytac MDBT50Q-1MV2 -> Raytac MDBT50Q-P1MV2
Changed lines of the file:
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@@
 			)
 		)
-		(property "Value" "MDBT50Q-1MV2"
+		(property "Value" "MDBT50Q-P1MV2"
 			(at 154.94 55.88 0)
 			(effects
@@
 			)
 		)
-		(property "LCSC" "C5118826"
+		(property "LCSC" "C5119772"
 			(at 154.94 55.88 0)
 			(hide yes)
@@
 			)
 		)
-		(property "MPN" "Raytac MDBT50Q-1MV2"
+		(property "MPN" "Raytac MDBT50Q-P1MV2"
 			(at 162.56 104.14 0)
 			(hide yes)
